Commit message: 0316-2重新修改了xacro文件，与launch文件，此状态可打开rviz与gazebo（仅小车）

File: install/agv_simulation/share/agv_simulation/description/robot.urdf.xacro (robot description, xacro)
@@ -1,177 +1 @@
-<?xml version="1.0"?>
-<robot name="my_agv" xmlns:xacro="http://www.ros.org/wiki/xacro">
-    <xacro:include filename="inertial_macros.xacro"/>
-    <material name="black"><color rgba="0 0 0 1"/></material>
-    <material name="white"><color rgba="1 1 1 1"/></material>
-    <material name="red"><color rgba="1 0 0 1"/></material>
-    <material name="blue"><color rgba="0 0 1 1"/></material>
-    <link name="base_footprint"/>
-    <joint name="base_joint" type="fixed">
-        <parent link="base_footprint"/>
-        <child link="base_link"/>
-        <origin xyz="0 0 0.05"/>
-    </joint>
-    <link name="base_link">
-        <visual>
-            <origin xyz="0 0 0.1"/>
-            <geometry>
-                <box size="0.4 0.3 0.2"/>
-            </geometry>
-            <material name="white"/>
-        </visual>
-        <collision>
-            <origin xyz="0 0 0.1"/>
-            <geometry>
-                <box size="0.4 0.3 0.2"/>
-            </geometry>
-        </collision>
-        <xacro:inertial_box mass="10.0" x="0.4" y="0.3" z="0.2">
-            <origin xyz="0 0 0.1" rpy="0 0 0"/>
-        </xacro:inertial_box>
-    </link>
-    <link name="lidar_link">
-        <visual>
-            <geometry>
-                <cylinder radius="0.05" length="0.04"/>
-            </geometry>
-            <material name="black"/>
-        </visual>
-        <xacro:inertial_cylinder mass="0.2" length="0.04" radius="0.05">
-            <origin xyz="0 0 0" rpy="0 0 0"/>
-        </xacro:inertial_cylinder>
-    </link>
-    <joint name="lidar_joint" type="fixed">
-        <parent link="base_link"/>
-        <child link="lidar_link"/>
-        <origin xyz="0 0 0.22" rpy="0 0 0"/>
-    </joint>
-    <gazebo reference="lidar_link">
-        <sensor name="lidar" type="ray">
-            <always_on>true</always_on>
-            <visualize>false</visualize> <update_rate>10</update_rate>
-            <ray>
-                <scan>
-                    <horizontal>
-                        <samples>440</samples>
-                        <resolution>1</resolution>
-                        <min_angle>-3.14159</min_angle>
-                        <max_angle>3.14159</max_angle>
-                    </horizontal>
-                    <vertical>
-                        <samples>16</samples>
-                        <resolution>1</resolution>
-                        <min_angle>-0.2617</min_angle> <max_angle>0.2617</max_angle>  </vertical>
-                </scan>
-                <range>
-                    <min>0.3</min>
-                    <max>12.0</max>
-                    <resolution>0.01</resolution>
-                </range>
-                <noise>
-                    <type>gaussian</type>
-                    <mean>0.0</mean>
-                    <stddev>0.01</stddev>
-                </noise>
-            </ray>
-            <plugin name="lidar_controller" filename="libgazebo_ros_ray_sensor.so">
-                <ros>
-                    <remapping>~/out:=/points_raw</remapping>
-                </ros>
-                <output_type>sensor_msgs/PointCloud2</output_type>
-                <frame_name>lidar_link</frame_name>
-            </plugin>
-        </sensor>
-    </gazebo>
-    <link name="camera_link">
-        <visual>
-            <geometry>
-                <box size="0.02 0.08 0.02"/>
-            </geometry>
-            <material name="red"/>
-        </visual>
-    </link>
-    <joint name="camera_joint" type="fixed">
-        <parent link="base_link"/>
-        <child link="camera_link"/>
-        <origin xyz="0.2 0 0.15" rpy="0 0 0"/>
-    </joint>
-    <link name="camera_link_optical"></link>
-    <joint name="camera_optical_joint" type="fixed">
-        <parent link="camera_link"/>
-        <child link="camera_link_optical"/>
-        <origin xyz="0 0 0" rpy="${-pi/2} 0 ${-pi/2}"/>
-    </joint>
-    <gazebo reference="camera_link">
-        <sensor name="camera" type="depth">
-            <visualize>true</visualize>
-            <update_rate>15</update_rate> <camera>
-                <horizontal_fov>1.089</horizontal_fov>
-                <image>
-                    <format>R8G8B8</format>
-                    <width>640</width>
-                    <height>480</height>
-                </image>
-                <clip>
-                    <near>0.1</near>
-                    <far>8.0</far>
-                </clip>
-            </camera>
-            <plugin name="camera_controller" filename="libgazebo_ros_camera.so">
-                <frame_name>camera_link_optical</frame_name>
-                <min_depth>0.1</min_depth>
-                <max_depth>8.0</max_depth>
-                <publish_point_cloud>true</publish_point_cloud>
-                <publish_depth_image>true</publish_depth_image>
-            </plugin>
-        </sensor>
-    </gazebo>
-    <link name="imu_link"/>
-    <joint name="imu_joint" type="fixed">
-        <parent link="base_link"/>
-        <child link="imu_link"/>
-        <origin xyz="0 0 0.1"/>
-    </joint>
-    <gazebo reference="imu_link">
-        <sensor name="imu_sensor" type="imu">
-            <plugin filename="libgazebo_ros_imu_sensor.so" name="imu_plugin">
-                <ros>
-                    <remapping>~/out:=/imu/data</remapping>
-                </ros>
-                <initial_orientation_as_reference>false</initial_orientation_as_reference>
-            </plugin>
-            <always_on>true</always_on>
-            <update_rate>100</update_rate>
-            <imu>
-                <noise>
-                    <type>gaussian</type>
-                    <rate>
-                        <mean>0.0</mean>
-                        <stddev>2e-4</stddev>
-                    </rate>
-                    <accel>
-                        <mean>0.0</mean>
-                        <stddev>1.7e-2</stddev>
-                    </accel>
-                </noise>
-            </imu>
-        </sensor>
-    </gazebo>
-    <gazebo>
-        <plugin name="diff_drive" filename="libgazebo_ros_diff_drive.so">
-            <ros>
-                <remapping>cmd_vel:=cmd_vel</remapping>
-                <remapping>odom:=odom</remapping>
-            </ros>
-            <left_joint>left_wheel_joint</left_joint> <right_joint>right_wheel_joint</right_joint>
-            <wheel_separation>0.35</wheel_separation>
-            <wheel_diameter>0.1</wheel_diameter>
-            <max_wheel_torque>20</max_wheel_torque>
-            <max_wheel_acceleration>1.0</max_wheel_acceleration>
-            <publish_odom>true</publish_odom>
-            <publish_odom_tf>true</publish_odom_tf>
-            <publish_wheel_tf>true</publish_wheel_tf>
-            <odometry_frame>odom</odometry_frame>
-            <robot_base_frame>base_footprint</robot_base_frame>
-        </plugin>
-    </gazebo>
-</robot>
+/home/lyq/bysj_ws/src/agv_simulation/description/robot.urdf.xacro

File: src/agv_simulation/description/robot.urdf.xacro (robot description, xacro)
@@ -1,177 +1,178 @@
 <?xml version="1.0"?>
-<robot name="my_agv" xmlns:xacro="http://www.ros.org/wiki/xacro">
-    <xacro:include filename="inertial_macros.xacro"/>
-    <material name="black"><color rgba="0 0 0 1"/></material>
-    <material name="white"><color rgba="1 1 1 1"/></material>
-    <material name="red"><color rgba="1 0 0 1"/></material>
-    <material name="blue"><color rgba="0 0 1 1"/></material>
-    <link name="base_footprint"/>
-    <joint name="base_joint" type="fixed">
-        <parent link="base_footprint"/>
-        <child link="base_link"/>
-        <origin xyz="0 0 0.05"/>
+<robot name="agv_bot" xmlns:xacro="http://www.ros.org/wiki/xacro">
+  <xacro:property name="base_width" value="0.4"/>
+  <xacro:property name="base_length" value="0.6"/>
+  <xacro:property name="base_height" value="0.2"/>
+  <xacro:property name="wheel_radius" value="0.1"/>
+  <xacro:property name="wheel_width" value="0.05"/>
+  <xacro:property name="wheel_ygap" value="0.05"/>
+  <xacro:property name="wheel_zoff" value="0.05"/>
+  <xacro:property name="wheel_xoff" value="0.15"/>
+  <material name="blue"> <color rgba="0 0 0.8 1"/> </material>
+  <material name="black"> <color rgba="0 0 0 1"/> </material>
+  <material name="gray"> <color rgba="0.5 0.5 0.5 1"/> </material>
+  <xacro:macro name="inertial_box" params="mass x y z">
+    <inertial>
+      <origin xyz="0 0 0" rpy="0 0 0"/>
+      <mass value="${mass}"/>
+      <inertia ixx="${(1/12) * mass * (y*y+z*z)}" ixy="0.0" ixz="0.0"
+               iyy="${(1/12) * mass * (x*x+z*z)}" iyz="0.0"
+               izz="${(1/12) * mass * (x*x+y*y)}"/>
+    </inertial>
+  </xacro:macro>
+  <xacro:macro name="inertial_cylinder" params="mass length radius">
+    <inertial>
+      <origin xyz="0 0 0" rpy="0 0 0"/>
+      <mass value="${mass}"/>
+      <inertia ixx="${(1/12) * mass * (3*radius*radius + length*length)}" ixy="0.0" ixz="0.0"
+               iyy="${(1/12) * mass * (3*radius*radius + length*length)}" iyz="0.0"
+               izz="${(1/2) * mass * (radius*radius)}"/>
+    </inertial>
+  </xacro:macro>
+  <link name="base_footprint"/>
+  <joint name="base_joint" type="fixed">
+    <parent link="base_footprint"/>
+    <child link="base_link"/>
+    <origin xyz="0 0 ${wheel_radius}" rpy="0 0 0"/>
+  </joint>
+  <link name="base_link">
+    <visual>
+      <geometry> <box size="${base_length} ${base_width} ${base_height}"/> </geometry>
+      <material name="blue"/>
+    </visual>
+    <collision>
+      <geometry> <box size="${base_length} ${base_width} ${base_height}"/> </geometry>
+    </collision>
+    <xacro:inertial_box mass="10.0" x="${base_length}" y="${base_width}" z="${base_height}"/>
+  </link>
+  <xacro:macro name="wheel" params="prefix x_reflect y_reflect">
+    <link name="${prefix}_wheel">
+      <visual>
+        <origin xyz="0 0 0" rpy="${pi/2} 0 0"/>
+        <geometry> <cylinder radius="${wheel_radius}" length="${wheel_width}"/> </geometry>
+        <material name="black"/>
+      </visual>
+      <collision>
+        <origin xyz="0 0 0" rpy="${pi/2} 0 0"/>
+        <geometry> <cylinder radius="${wheel_radius}" length="${wheel_width}"/> </geometry>
+      </collision>
+      <xacro:inertial_cylinder mass="0.5" length="${wheel_width}" radius="${wheel_radius}"/>
+    </link>
+    <joint name="${prefix}_wheel_joint" type="continuous">
+      <parent link="base_link"/>
+      <child link="${prefix}_wheel"/>
+      <origin xyz="${x_reflect*wheel_xoff} ${y_reflect*(base_width/2+wheel_ygap)} ${-wheel_zoff}" rpy="0 0 0"/>
+      <axis xyz="0 1 0"/>
     </joint>
-    <link name="base_link">
-        <visual>
-            <origin xyz="0 0 0.1"/>
-            <geometry>
-                <box size="0.4 0.3 0.2"/>
-            </geometry>
-            <material name="white"/>
-        </visual>
-        <collision>
-            <origin xyz="0 0 0.1"/>
-            <geometry>
-                <box size="0.4 0.3 0.2"/>
-            </geometry>
-        </collision>
-        <xacro:inertial_box mass="10.0" x="0.4" y="0.3" z="0.2">
-            <origin xyz="0 0 0.1" rpy="0 0 0"/>
-        </xacro:inertial_box>
-    </link>
-    <link name="lidar_link">
-        <visual>
-            <geometry>
-                <cylinder radius="0.05" length="0.04"/>
-            </geometry>
-            <material name="black"/>
-        </visual>
-        <xacro:inertial_cylinder mass="0.2" length="0.04" radius="0.05">
-            <origin xyz="0 0 0" rpy="0 0 0"/>
-        </xacro:inertial_cylinder>
-    </link>
-    <joint name="lidar_joint" type="fixed">
-        <parent link="base_link"/>
-        <child link="lidar_link"/>
-        <origin xyz="0 0 0.22" rpy="0 0 0"/>
-    </joint>
-    <gazebo reference="lidar_link">
-        <sensor name="lidar" type="ray">
-            <always_on>true</always_on>
-            <visualize>false</visualize> <update_rate>10</update_rate>
-            <ray>
-                <scan>
-                    <horizontal>
-                        <samples>440</samples>
-                        <resolution>1</resolution>
-                        <min_angle>-3.14159</min_angle>
-                        <max_angle>3.14159</max_angle>
-                    </horizontal>
-                    <vertical>
-                        <samples>16</samples>
-                        <resolution>1</resolution>
-                        <min_angle>-0.2617</min_angle> <max_angle>0.2617</max_angle>  </vertical>
-                </scan>
-                <range>
-                    <min>0.3</min>
-                    <max>12.0</max>
-                    <resolution>0.01</resolution>
-                </range>
-                <noise>
-                    <type>gaussian</type>
-                    <mean>0.0</mean>
-                    <stddev>0.01</stddev>
-                </noise>
-            </ray>
-            <plugin name="lidar_controller" filename="libgazebo_ros_ray_sensor.so">
-                <ros>
-                    <remapping>~/out:=/points_raw</remapping>
-                </ros>
-                <output_type>sensor_msgs/PointCloud2</output_type>
-                <frame_name>lidar_link</frame_name>
-            </plugin>
-        </sensor>
-    </gazebo>
-    <link name="camera_link">
-        <visual>
-            <geometry>
-                <box size="0.02 0.08 0.02"/>
-            </geometry>
-            <material name="red"/>
-        </visual>
-    </link>
-    <joint name="camera_joint" type="fixed">
-        <parent link="base_link"/>
-        <child link="camera_link"/>
-        <origin xyz="0.2 0 0.15" rpy="0 0 0"/>
-    </joint>
-    <link name="camera_link_optical"></link>
-    <joint name="camera_optical_joint" type="fixed">
-        <parent link="camera_link"/>
-        <child link="camera_link_optical"/>
-        <origin xyz="0 0 0" rpy="${-pi/2} 0 ${-pi/2}"/>
-    </joint>
-    <gazebo reference="camera_link">
-        <sensor name="camera" type="depth">
-            <visualize>true</visualize>
-            <update_rate>15</update_rate> <camera>
-                <horizontal_fov>1.089</horizontal_fov>
-                <image>
-                    <format>R8G8B8</format>
-                    <width>640</width>
-                    <height>480</height>
-                </image>
-                <clip>
-                    <near>0.1</near>
-                    <far>8.0</far>
-                </clip>
-            </camera>
-            <plugin name="camera_controller" filename="libgazebo_ros_camera.so">
-                <frame_name>camera_link_optical</frame_name>
-                <min_depth>0.1</min_depth>
-                <max_depth>8.0</max_depth>
-                <publish_point_cloud>true</publish_point_cloud>
-                <publish_depth_image>true</publish_depth_image>
-            </plugin>
-        </sensor>
-    </gazebo>
-    <link name="imu_link"/>
-    <joint name="imu_joint" type="fixed">
-        <parent link="base_link"/>
-        <child link="imu_link"/>
-        <origin xyz="0 0 0.1"/>
-    </joint>
-    <gazebo reference="imu_link">
-        <sensor name="imu_sensor" type="imu">
-            <plugin filename="libgazebo_ros_imu_sensor.so" name="imu_plugin">
-                <ros>
-                    <remapping>~/out:=/imu/data</remapping>
-                </ros>
-                <initial_orientation_as_reference>false</initial_orientation_as_reference>
-            </plugin>
-            <always_on>true</always_on>
-            <update_rate>100</update_rate>
-            <imu>
-                <noise>
-                    <type>gaussian</type>
-                    <rate>
-                        <mean>0.0</mean>
-                        <stddev>2e-4</stddev>
-                    </rate>
-                    <accel>
-                        <mean>0.0</mean>
-                        <stddev>1.7e-2</stddev>
-                    </accel>
-                </noise>
-            </imu>
-        </sensor>
-    </gazebo>
-    <gazebo>
-        <plugin name="diff_drive" filename="libgazebo_ros_diff_drive.so">
-            <ros>
-                <remapping>cmd_vel:=cmd_vel</remapping>
-                <remapping>odom:=odom</remapping>
-            </ros>
-            <left_joint>left_wheel_joint</left_joint> <right_joint>right_wheel_joint</right_joint>
-            <wheel_separation>0.35</wheel_separation>
-            <wheel_diameter>0.1</wheel_diameter>
-            <max_wheel_torque>20</max_wheel_torque>
-            <max_wheel_acceleration>1.0</max_wheel_acceleration>
-            <publish_odom>true</publish_odom>
-            <publish_odom_tf>true</publish_odom_tf>
-            <publish_wheel_tf>true</publish_wheel_tf>
-            <odometry_frame>odom</odometry_frame>
-            <robot_base_frame>base_footprint</robot_base_frame>
-        </plugin>
-    </gazebo>
+  </xacro:macro>
+  <xacro:wheel prefix="drivewhl_l" x_reflect="-1" y_reflect="1" />
+  <xacro:wheel prefix="drivewhl_r" x_reflect="-1" y_reflect="-1" />
+  <link name="front_caster">
+    <visual>
+      <geometry> <sphere radius="${wheel_radius/2}"/> </geometry>
+      <material name="gray"/>
+    </visual>
+    <collision>
+      <geometry> <sphere radius="${wheel_radius/2}"/> </geometry>
+    </collision>
+    <xacro:inertial_cylinder mass="0.2" length="0.05" radius="${wheel_radius/2}"/>
+  </link>
+  <joint name="caster_joint" type="fixed">
+    <parent link="base_link"/>
+    <child link="front_caster"/>
+    <origin xyz="${wheel_xoff} 0 ${-wheel_zoff - wheel_radius/2}" rpy="0 0 0"/>
+  </joint>
+  <link name="laser_link">
+    <visual>
+      <geometry> <cylinder radius="0.05" length="0.08"/> </geometry>
+      <material name="gray"/>
+    </visual>
+    <xacro:inertial_cylinder mass="0.1" length="0.08" radius="0.05"/>
+  </link>
+  <joint name="laser_joint" type="fixed">
+    <parent link="base_link"/>
+    <child link="laser_link"/>
+    <origin xyz="0.1 0 ${base_height/2 + 0.04}" rpy="0 0 0"/>
+  </joint>
+  <link name="imu_link">
+    <xacro:inertial_box mass="0.01" x="0.01" y="0.01" z="0.01"/>
+  </link>
+  <joint name="imu_joint" type="fixed">
+    <parent link="base_link"/>
+    <child link="imu_link"/>
+    <origin xyz="0 0 0" rpy="0 0 0"/>
+  </joint>
+  <link name="camera_link">
+    <visual>
+      <geometry> <box size="0.02 0.1 0.03"/> </geometry>
+    </visual>
+    <xacro:inertial_box mass="0.05" x="0.02" y="0.1" z="0.03"/>
+  </link>
+  <joint name="camera_joint" type="fixed">
+    <parent link="base_link"/>
+    <child link="camera_link"/>
+    <origin xyz="${base_length/2} 0 0.05" rpy="0 0 0"/>
+  </joint>
+  <gazebo>
+    <plugin name='diff_drive' filename='libgazebo_ros_diff_drive.so'>
+      <ros> <namespace>/</namespace> </ros>
+      <left_joint>drivewhl_l_wheel_joint</left_joint>
+      <right_joint>drivewhl_r_wheel_joint</right_joint>
+      <wheel_separation>${base_width + 2*wheel_ygap}</wheel_separation>
+      <wheel_diameter>${2*wheel_radius}</wheel_diameter>
+      <publish_odom>true</publish_odom>
+      <publish_odom_tf>true</publish_odom_tf>
+      <publish_wheel_tf>true</publish_wheel_tf>
+      <odometry_frame>odom</odometry_frame>
+      <robot_base_frame>base_footprint</robot_base_frame>
+      <max_wheel_torque>200</max_wheel_torque>
+      <max_wheel_acceleration>10.0</max_wheel_acceleration>
+    </plugin>
+  </gazebo>
+  <gazebo reference="laser_link">
+    <sensor name="3d_lidar" type="ray">
+      <always_on>true</always_on>
+      <visualize>false</visualize>
+      <update_rate>10</update_rate>
+      <ray>
+        <scan>
+          <horizontal>
+            <samples>360</samples>
+            <resolution>1</resolution>
+            <min_angle>-3.14</min_angle>
+            <max_angle>3.14</max_angle>
+          </horizontal>
+          <vertical>
+            <samples>16</samples>
+            <resolution>1</resolution>
+            <min_angle>-0.26</min_angle>
+            <max_angle>0.26</max_angle>
+          </vertical>
+        </scan>
+        <range>
+          <min>0.3</min>
+          <max>12.0</max>
+          <resolution>0.01</resolution>
+        </range>
+      </ray>
+      <plugin name="lidar_plugin" filename="libgazebo_ros_ray_sensor.so">
+        <ros>
+          <remapping>~/out:=scan_3d</remapping>
+        </ros>
+        <output_type>sensor_msgs/PointCloud2</output_type>
+        <frame_name>laser_link</frame_name>
+      </plugin>
+    </sensor>
+  </gazebo>
+  <gazebo reference="imu_link">
+    <sensor name="imu_sensor" type="imu">
+      <always_on>true</always_on>
+      <update_rate>100</update_rate>
+      <plugin name="imu_plugin" filename="libgazebo_ros_imu_sensor.so">
+        <ros>
+          <remapping>~/out:=imu</remapping>
+        </ros>
+      </plugin>
+    </sensor>
+  </gazebo>
 </robot>
