Commit message: 0316-3更新了摄像头点云空间配准问题，此版本能仿真出小车和world（仅红色方块）

File: src/agv_simulation/description/robot.urdf.xacro (robot description, xacro)
@@ -114,4 +114,27 @@
     <origin xyz="${base_length/2} 0 0.05" rpy="0 0 0"/>
   </joint>
+  <link name="camera_link_optical"></link>
+  <joint name="camera_optical_joint" type="fixed">
+    <parent link="camera_link"/>
+    <child link="camera_link_optical"/>
+    <origin xyz="0 0 0" rpy="${-pi/2} 0 ${-pi/2}"/>
+  </joint>
+  <gazebo reference="base_link">
+    <material>Gazebo/Blue</material>
+  </gazebo>
+  <gazebo reference="drivewhl_l_wheel">
+    <material>Gazebo/Black</material>
+  </gazebo>
+  <gazebo reference="drivewhl_r_wheel">
+    <material>Gazebo/Black</material>
+  </gazebo>
+  <gazebo reference="front_caster">
+    <material>Gazebo/Grey</material>
+    <mu1 value="0.001"/>
+    <mu2 value="0.001"/>
+  </gazebo>
+  <gazebo reference="laser_link">
+    <material>Gazebo/Black</material>
+  </gazebo>
   <gazebo>
     <plugin name='diff_drive' filename='libgazebo_ros_diff_drive.so'>
@@ -176,3 +199,30 @@
     </sensor>
   </gazebo>
+  <gazebo reference="camera_link">
+    <sensor name="depth_camera" type="depth">
+      <visualize>true</visualize>
+      <update_rate>30.0</update_rate>
+      <camera name="camera">
+        <horizontal_fov>1.047</horizontal_fov>
+        <image>
+          <width>640</width>
+          <height>480</height>
+          <format>R8G8B8</format>
+        </image>
+        <clip>
+          <near>0.05</near>
+          <far>3.0</far>
+        </clip>
+     </camera>
+      <plugin name="camera_controller" filename="libgazebo_ros_camera.so">
+        <ros>
+          <remapping>depth/image_raw:=depth_image</remapping>
+          <remapping>points:=camera_points</remapping>
+        </ros>
+        <frame_name>camera_link_optical</frame_name>
+        <min_depth>0.1</min_depth>
+        <max_depth>10.0</max_depth>
+      </plugin>
+    </sensor>
+  </gazebo>
 </robot>

Commit message: 更新了ekf融合里程计和IMU，此版本 尚有疑问，但ros2 topic echo /odometry/filtered有数据输出

File: src/agv_simulation/description/robot.urdf.xacro (robot description, xacro)
@@ -31,8 +31,8 @@
   </xacro:macro>
   <link name="base_footprint"/>
-  <joint name="base_joint" type="fixed">
+  <joint name="base_footprint_joint" type="fixed">
     <parent link="base_footprint"/>
     <child link="base_link"/>
-    <origin xyz="0 0 ${wheel_radius}" rpy="0 0 0"/>
+    <origin xyz="0 0 0.1" rpy="0 0 0"/>
   </joint>
   <link name="base_link">
@@ -145,7 +145,7 @@
       <wheel_diameter>${2*wheel_radius}</wheel_diameter>
       <publish_odom>true</publish_odom>
-      <publish_odom_tf>true</publish_odom_tf>
+      <publish_odom_tf>false</publish_odom_tf>
       <publish_wheel_tf>true</publish_wheel_tf>
-      <odometry_frame>odom</odometry_frame>
+      <odometry_frame>odom_raw</odometry_frame>
       <robot_base_frame>base_footprint</robot_base_frame>
       <max_wheel_torque>200</max_wheel_torque>
